File: Projet_Tschema/Projet_Tschema.kicad_sch (KiCad schematic)
At the start: 41 parts, among them J1 Raspberry_Pi_2_3, J2 Screw_Terminal_01x02, J3 Conn_D42V55F5, U1 SC16IS-752, U2 AMS1117, Y1 14.7456M

Commit message: pcb
Parts:
- C4, C5: footprint (none) -> Capacitor_SMD:C_0805_2012Metric
- J2: footprint (none) -> Connector_PinHeader_2.54mm:PinHeader_1x02_P2.54mm_Vertical
- J3: footprint (none) -> Connector_PinHeader_2.54mm:PinHeader_2x06_P2.54mm_Vertical
Changed lines of the file:
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@@
 			)
 		)
-		(property "Footprint" ""
+		(property "Footprint" "Capacitor_SMD:C_0805_2012Metric"
 			(at 232.41 113.03 0)
 			(effects
@@
 			)
 		)
-		(property "Footprint" ""
+		(property "Footprint" "Connector_PinHeader_2.54mm:PinHeader_1x02_P2.54mm_Vertical"
 			(at 166.37 139.7 0)
 			(effects
@@
 			)
 		)
-		(property "Footprint" ""
+		(property "Footprint" "Capacitor_SMD:C_0805_2012Metric"
 			(at 207.01 113.03 0)
 			(effects
@@
 			)
 		)
-		(property "Footprint" ""
+		(property "Footprint" "Connector_PinHeader_2.54mm:PinHeader_2x06_P2.54mm_Vertical"
 			(at 166.37 109.22 0)
 			(effects

Commit message: first version finished
Parts:
- removed D2: LED_Filled, LED_SMD:LED_0805_2012Metric, symbol Device:LED_Filled
- removed R14, R15, R16, R17, R18, R19, R20, R21, R22, R23: NC, Resistor_SMD:R_0805_2012Metric, symbol Device:R_US
- removed R24: 1K, Resistor_SMD:R_0805_2012Metric, symbol Device:R_US
- Y1: footprint Crystal:Crystal_SMD_3225-4Pin_3.2x2.5mm -> Crystal:Crystal_HC52-U_Vertical
Connections:
- net 5V: now also J3.11 (Pin_11); no longer J3.6 (Pin_6)
- net GND: now also J3.7 (Pin_7), J3.8 (Pin_8), J3.9 (Pin_9); no longer J3.11 (Pin_11), J3.4 (Pin_4), J3.5 (Pin_5)
- net Vin: now also J3.5 (Pin_5), J3.6 (Pin_6); no longer J3.3 (Pin_3), J3.9 (Pin_9)
- net CTSA: no longer names the net of U1.2 (~{CTSA})
- net CTSA: no longer H1.6 (Pin_6)
- net CTSB: no longer names the net of U1.16 (~{CTSB})
- net CTSB: no longer H2.6 (Pin_6)
- net P20: no longer names the net of J1.38 (GPIO28)
- net P21: no longer names the net of J1.40 (GPIO29)
- net P22: no longer names the net of J1.15 (GPIO3)
- net P23: no longer names the net of J1.16 (GPIO4)
- net RTSA: no longer names the net of U1.1 (~{RTSA})
- net RTSA: no longer H1.5 (Pin_5)
- net RTSB: no longer names the net of U1.17 (~{RTSB})
- net RTSB: no longer H2.5 (Pin_5)
- no-connect marks 35 -> 48
Other:
- moved on the sheet: R11, R12, R13

Commit message: routes updated
Parts:
- removed J3: Conn_D42V55F5, Connector_PinHeader_2.54mm:PinHeader_2x06_P2.54mm_Vertical, symbol Connector_Generic:Conn_02x06_Top_Bottom
- added J3: DRF0571_Vout, Connector_PinHeader_2.54mm:PinHeader_1x01_P2.54mm_Vertical, symbol Connector_Generic:Conn_01x01
- added J4: DRF0571_Vin-, Connector_PinHeader_2.54mm:PinHeader_1x01_P2.54mm_Vertical, symbol Connector_Generic:Conn_01x01
- added J5: DRF0571_Vin, Connector_PinHeader_2.54mm:PinHeader_1x01_P2.54mm_Vertical, symbol Connector_Generic:Conn_01x01
- added J6: DRF0571_Vout-, Connector_PinHeader_2.54mm:PinHeader_1x01_P2.54mm_Vertical, symbol Connector_Generic:Conn_01x01
Connections:
- net 5V: now also J3.1 (Pin_1)
- net GND: now also J4.1 (Pin_1), J6.1 (Pin_1)
- net Vin: now also J5.1 (Pin_1)
- no-connect marks 48 -> 44
